File: ArmElectronics/ArmElectronics.sch (KiCad schematic (older format))
At the start: 3 parts

Commit message: Added in Pololu2581
Parts:
- added U?: Pololu_2851, symbol AidenMiniLibrary:Pololu_2851
Changed lines of the file:
@@
+	1    0    0    -1
+$EndComp
+$Comp
+L AidenMiniLibrary:Pololu_2851 U?
+U 1 1 5F72D60A
+P 8300 1700
+F 0 "U?" H 8258 2325 50  0000 C CNN
+F 1 "Pololu_2851" H 8258 2234 50  0000 C CNN
+F 2 "" H 8200 1500 50  0001 C CNN
+F 3 "" H 8200 1500 50  0001 C CNN
+	1    8300 1700
 	1    0    0    -1
 $EndComp

Commit message: Fixed a weird error
Parts:
- added U?: Teensy4.1, symbol ArmElectronics_Library:Teensy4.1
Changed lines of the file:
@@
+	1    0    0    -1
+$EndComp
+$Comp
+L ArmElectronics_Library:Teensy4.1 U?
+U 1 1 5F72F20F
+P 2250 4900
+F 0 "U?" H 2200 5615 50  0000 C CNN
+F 1 "Teensy4.1" H 2200 5524 50  0000 C CNN
+F 2 "" H 2100 4900 50  0001 C CNN
+F 3 "" H 2100 4900 50  0001 C CNN
+	1    2250 4900
 	1    0    0    -1
 $EndComp

Commit message: Finished motor drivers and motors
(Not connected to teensy)
Parts:
- added U? (x3): PA-09, symbol ArmElectronics_Library:PA-09
- added U? (x3): TB9051FTG, symbol ArmElectronics_Library:TB9051FTG
- added U?: Pololu_2857, symbol ArmElectronics_Library:Pololu_2857
- U?: symbol AidenMiniLibrary:Pololu_2851 -> ArmElectronics-rescue:Pololu_2851-AidenMiniLibrary
Connections:
- net labels added: +12V, +5V, GND, M1_DIAG, M1_HALL1, M1_HALL2, M1_OCM, M1_PWM1, M1_PWM2, M2_DIAG, M2_HALL1, M2_HALL2, M2_OCM, M2_PWM1, M2_PWM2, M3_DIAG, M3_HALL1, M3_HALL2, M3_OCM, M3_PWM1, M3_PWM2
- wire segments 0 -> 75
- no-connect marks 0 -> 15
Other:
- moved on the sheet: J?

Commit message: Little cleanup
Parts:
- removed U?: Pololu_2851, symbol ArmElectronics-rescue:Pololu_2851-AidenMiniLibrary
- added U?: Pololu_2851, symbol ArmElectronics_Library:Pololu_2851
Changed lines of the file:
@@
-$EndComp
-$Comp
-L ArmElectronics-rescue:Pololu_2851-AidenMiniLibrary U?
-U 1 1 5F72D60A
-P 6350 3950
-F 0 "U?" H 6308 4575 50  0000 C CNN
-F 1 "Pololu_2851" H 6308 4484 50  0000 C CNN
-F 2 "" H 6250 3750 50  0001 C CNN
-F 3 "" H 6250 3750 50  0001 C CNN
-	1    6350 3950
-	1    0    0    -1
 $EndComp
 $Comp
@@
 Wire Wire Line
 	15050 4500 15150 4500
+$Comp
+L ArmElectronics_Library:Pololu_2851 U?
+U 1 1 5F880EAA
+P 6350 2950
+F 0 "U?" H 6308 3575 50  0000 C CNN
+F 1 "Pololu_2851" H 6308 3484 50  0000 C CNN
+F 2 "" H 6250 2750 50  0001 C CNN
+F 3 "" H 6250 2750 50  0001 C CNN
+	1    6350 2950
+	1    0    0    -1
+$EndComp
 $EndSCHEMATC

Commit message: Power section
Connections:
- net +12V: now also J?.1 (Pin_1), U?.2 (VIN), U?.3 (VIN)
- net +5V: now also U?.5 (Vout)
- net GND: now also J?.2 (Pin_2), U?.3 (GND), U?.4 (GND), U?.4 (GND), U?.6 (GND)
- net +3V3: now reaches U?.5 (VOUT)
- no-connect marks 15 -> 18
Other:
- moved on the sheet: J?, U?
Changed lines of the file:
@@
 L Connector_Generic:Conn_01x02 J?
 U 1 1 5F72C87F
-P 5350 3550
-F 0 "J?" H 5430 3542 50  0000 L CNN
-F 1 "Power In" H 5430 3451 50  0000 L CNN
-F 2 "" H 5350 3550 50  0001 C CNN
-F 3 "~" H 5350 3550 50  0001 C CNN
-	1    5350 3550
+P 9500 1100
+F 0 "J?" H 9580 1092 50  0000 L CNN
+F 1 "Power In" H 9580 1001 50  0000 L CNN
+F 2 "" H 9500 1100 50  0001 C CNN
+F 3 "~" H 9500 1100 50  0001 C CNN
+	1    9500 1100
 	1    0    0    -1
 $EndComp
@@
 L ArmElectronics_Library:Pololu_2857 U?
 U 1 1 5F85182A
-P 8400 3500
-F 0 "U?" H 8400 3575 50  0000 C CNN
-F 1 "Pololu_2857" H 8400 3484 50  0000 C CNN
-F 2 "" H 8400 3500 50  0001 C CNN
-F 3 "" H 8400 3500 50  0001 C CNN
-	1    8400 3500
+P 9300 2050
+F 0 "U?" H 9300 2125 50  0000 C CNN
+F 1 "Pololu_2857" H 9300 2034 50  0000 C CNN
+F 2 "" H 9300 2050 50  0001 C CNN
+F 3 "" H 9300 2050 50  0001 C CNN
+	1    9300 2050
 	1    0    0    -1
 $EndComp
@@
 L ArmElectronics_Library:Pololu_2851 U?
 U 1 1 5F880EAA
-P 6350 2950
-F 0 "U?" H 6308 3575 50  0000 C CNN
-F 1 "Pololu_2851" H 6308 3484 50  0000 C CNN
-F 2 "" H 6250 2750 50  0001 C CNN
-F 3 "" H 6250 2750 50  0001 C CNN
-	1    6350 2950
-	1    0    0    -1
-$EndComp
+P 9400 3500
+F 0 "U?" H 9358 4125 50  0000 C CNN
+F 1 "Pololu_2851" H 9358 4034 50  0000 C CNN
+F 2 "" H 9300 3300 50  0001 C CNN
+F 3 "" H 9300 3300 50  0001 C CNN
+	1    9400 3500
+	1    0    0    -1
+$EndComp
+$Comp
+L power:GND #PWR?
+U 1 1 5F884274
+P 9150 1200
+F 0 "#PWR?" H 9150 950 50  0001 C CNN
+F 1 "GND" H 9155 1027 50  0000 C CNN
+F 2 "" H 9150 1200 50  0001 C CNN
+F 3 "" H 9150 1200 50  0001 C CNN
+	1    9150 1200
+	1    0    0    -1
+$EndComp
+$Comp
+L power:+12V #PWR?
+U 1 1 5F884B1A
+P 9150 1100
+F 0 "#PWR?" H 9150 950 50  0001 C CNN
+F 1 "+12V" H 9165 1273 50  0000 C CNN
+F 2 "" H 9150 1100 50  0001 C CNN
+F 3 "" H 9150 1100 50  0001 C CNN
+	1    9150 1100
+	1    0    0    -1
+$EndComp
+Wire Wire Line
+	9150 1100 9300 1100
+Wire Wire Line
+	9300 1200 9150 1200
+$Comp
+L power:+12V #PWR?
+U 1 1 5F889DBE
+P 8600 2400
+F 0 "#PWR?" H 8600 2250 50  0001 C CNN
+F 1 "+12V" H 8615 2573 50  0000 C CNN
+F 2 "" H 8600 2400 50  0001 C CNN
+F 3 "" H 8600 2400 50  0001 C CNN
+	1    8600 2400
+	1    0    0    -1
+$EndComp
+Wire Wire Line
+	8600 2400 8950 2400
+$Comp
+L power:GND #PWR?
+U 1 1 5F88CA48
+P 8600 2500
+F 0 "#PWR?" H 8600 2250 50  0001 C CNN
+F 1 "GND" H 8605 2327 50  0000 C CNN
+F 2 "" H 8600 2500 50  0001 C CNN
+F 3 "" H 8600 2500 50  0001 C CNN
+	1    8600 2500
+	1    0    0    -1
+$EndComp
+Wire Wire Line
+	8600 2500 8950 2500
+$Comp
+L power:+3.3V #PWR?
+U 1 1 5F88F76F
+P 9850 2200
+F 0 "#PWR?" H 9850 2050 50  0001 C CNN
+F 1 "+3.3V" H 9865 2373 50  0000 C CNN
+F 2 "" H 9850 2200 50  0001 C CNN
+F 3 "" H 9850 2200 50  0001 C CNN
+	1    9850 2200
+	1    0    0    -1
+$EndComp
+Wire Wire Line
+	9850 2200 9650 2200
+$Comp
+L power:GND #PWR?
+U 1 1 5F893080
+P 9850 2300
+F 0 "#PWR?" H 9850 2050 50  0001 C CNN
+F 1 "GND" H 9855 2127 50  0000 C CNN
+F 2 "" H 9850 2300 50  0001 C CNN
+F 3 "" H 9850 2300 50  0001 C CNN
+	1    9850 2300
+	1    0    0    -1
+$EndComp
+Wire Wire Line
+	9850 2300 9650 2300
+NoConn ~ 8950 2300
+NoConn ~ 8950 2200
+$Comp
+L power:+12V #PWR?
+U 1 1 5F89AD29
+P 9950 3400
+F 0 "#PWR?" H 9950 3250 50  0001 C CNN
+F 1 "+12V" H 9965 3573 50  0000 C CNN
+F 2 "" H 9950 3400 50  0001 C CNN
+F 3 "" H 9950 3400 50  0001 C CNN
+	1    9950 3400
+	1    0    0    -1
+$EndComp
+Wire Wire Line
+	9950 3400 9700 3400
+$Comp
+L power:GND #PWR?
+U 1 1 5F89DC47
+P 9850 3600
+F 0 "#PWR?" H 9850 3350 50  0001 C CNN
+F 1 "GND" H 9855 3427 50  0000 C CNN
+F 2 "" H 9850 3600 50  0001 C CNN
+F 3 "" H 9850 3600 50  0001 C CNN
+	1    9850 3600
+	1    0    0    -1
+$EndComp
+Wire Wire Line
+	9850 3600 9850 3300
+Wire Wire Line
+	9850 3200 9700 3200
+Wire Wire Line
+	9700 3300 9850 3300
+Connection ~ 9850 3300
+Wire Wire Line
+	9850 3300 9850 3200
+NoConn ~ 9700 3500
+$Comp
+L power:+5V #PWR?
+U 1 1 5F8A6B13
+P 9950 3100
+F 0 "#PWR?" H 9950 2950 50  0001 C CNN
+F 1 "+5V" H 9965 3273 50  0000 C CNN
+F 2 "" H 9950 3100 50  0001 C CNN
+F 3 "" H 9950 3100 50  0001 C CNN
+	1    9950 3100
+	1    0    0    -1
+$EndComp
+Wire Wire Line
+	9950 3100 9700 3100
 $EndSCHEMATC

Commit message: forgot that connecting different logic voltages together lets the magic smoke out
Parts:
- added Q1, Q10, Q11, Q12, Q13, Q14, Q15, Q16, Q17, Q18, Q2, Q3, Q4, Q5, Q6, Q7, Q8, Q9: Q_NMOS_DGS, symbol Device:Q_NMOS_DGS
- added R1, R10, R11, R12, R13, R14, R15, R16, R17, R18, R19, R2, R20, R21, R22, R23, R24, R25, R26, R27, R28, R29, R3, R30, R31, R32, R33, R34, R35, R36, R4, R5, R6, R7, R8, R9: 10k, symbol Device:R_Small
- gave numbers to parts that had none: 12
Connections:
- net +3V3: now also Q1.2 (G), Q10.2 (G), Q11.2 (G), Q12.2 (G), Q13.2 (G), Q14.2 (G), Q15.2 (G), Q16.2 (G), Q17.2 (G), Q18.2 (G), Q2.2 (G), Q3.2 (G), Q4.2 (G), Q5.2 (G), Q6.2 (G), Q7.2 (G), Q8.2 (G), Q9.2 (G), R1.2, R13.2, R14.2, R15.2, R16.2, R17.2, R18.2, R2.2, R25.2, R26.2, R27.2, R28.2, R29.2, R3.2, R30.2, R4.2, R5.2, R6.2
- net +5V: now also R10.1, R11.1, R12.1, R19.1, R20.1, R21.1, R22.1, R23.1, R24.1, R31.1, R32.1, R33.1, R34.1, R35.1, R36.1, R7.1, R8.1, R9.1
- net M1_DIAG: now also Q4.1 (D), R10.2
- net M1_HALL1: now also Q5.1 (D), R11.2
- net M1_HALL2: now also Q6.1 (D), R12.2
- net M1_OCM: now also Q3.1 (D), R9.2
- net M1_PWM1: now also Q1.1 (D), R7.2
- net M1_PWM2: now also Q2.1 (D), R8.2
- net M2_DIAG: now also Q10.1 (D), R22.2
- net M2_HALL1: now also Q11.1 (D), R23.2
- net M2_HALL2: now also Q12.1 (D), R24.2
- net M2_OCM: now also Q9.1 (D), R21.2
- net M2_PWM1: now also Q7.1 (D), R19.2
- net M2_PWM2: now also Q8.1 (D), R20.2
- net M3_DIAG: now also Q16.1 (D), R34.2
- net M3_HALL1: now also Q17.1 (D), R35.2
- net M3_HALL2: now also Q18.1 (D), R36.2
- net M3_OCM: now also Q15.1 (D), R33.2
- net M3_PWM1: now also Q13.1 (D), R31.2
- net M3_PWM2: now also Q14.1 (D), R32.2
- new net M1_DIAG_3v: Q4.3 (S), R4.1
- new net M1_HALL1_3v: Q5.3 (S), R5.1
- new net M1_HALL2_3v: Q6.3 (S), R6.1
- new net M1_OCM_3v: Q3.3 (S), R3.1
- new net M1_PWM1_3v: Q1.3 (S), R1.1
- new net M1_PWM2_3v: Q2.3 (S), R2.1
- new net M2_DIAG_3v: Q10.3 (S), R16.1
- new net M2_HALL1_3v: Q11.3 (S), R17.1
- new net M2_HALL2_3v: Q12.3 (S), R18.1
- new net M2_OCM_3v: Q9.3 (S), R15.1
- new net M2_PWM1_3v: Q7.3 (S), R13.1
- new net M2_PWM2_3v: Q8.3 (S), R14.1
- new net M3_DIAG_3v: Q16.3 (S), R28.1
- new net M3_HALL1_3v: Q17.3 (S), R29.1
- new net M3_HALL2_3v: Q18.3 (S), R30.1
- new net M3_OCM_3v: Q15.3 (S), R27.1
- new net M3_PWM1_3v: Q13.3 (S), R25.1
- new net M3_PWM2_3v: Q14.3 (S), R26.1
Other:
- moved on the sheet: U1, U4

Commit message: Small changes
Parts:
- Q1, Q10, Q11, Q12, Q13, Q14, Q15, Q16, Q17, Q18, Q2, Q3, Q4, Q5, Q6, Q7, Q8, Q9: value Q_NMOS_DGS -> BSS138
Connections:
- net +3V3: now also U4.1 (VIN)
- net GND: now also U4.3 (GND)
- net RPi_SDA: now reaches J1.3 (SDA/GPIO2)
- net RPi_SDA: now also U4.4 (SDA)
- net RPi_SCL: now reaches J1.5 (SCL/GPIO3)
- net RPi_SCL: now also U4.5 (SCL)
- net BNO055_RST: now reaches J1.7 (GCLK0/GPIO4)
- net BNO055_RST: now also U4.6 (RST)
- no-connect marks 18 -> 23
Changed lines of the file:
@@
 P 17400 1400
 F 0 "Q1" V 17649 1400 50  0000 C CNN
-F 1 "Q_NMOS_DGS" V 17740 1400 50  0000 C CNN
+F 1 "BSS138" V 17740 1400 50  0000 C CNN
 F 2 "" H 17600 1500 50  0001 C CNN
 F 3 "~" H 17400 1400 50  0001 C CNN
@@
 P 17400 2400
 F 0 "Q2" V 17649 2400 50  0000 C CNN
-F 1 "Q_NMOS_DGS" V 17740 2400 50  0000 C CNN
+F 1 "BSS138" V 17740 2400 50  0000 C CNN
 F 2 "" H 17600 2500 50  0001 C CNN
 F 3 "~" H 17400 2400 50  0001 C CNN
@@
 P 17400 3400
 F 0 "Q3" V 17649 3400 50  0000 C CNN
-F 1 "Q_NMOS_DGS" V 17740 3400 50  0000 C CNN
+F 1 "BSS138" V 17740 3400 50  0000 C CNN
 F 2 "" H 17600 3500 50  0001 C CNN
 F 3 "~" H 17400 3400 50  0001 C CNN
@@
 P 17400 4400
 F 0 "Q4" V 17649 4400 50  0000 C CNN
-F 1 "Q_NMOS_DGS" V 17740 4400 50  0000 C CNN
+F 1 "BSS138" V 17740 4400 50  0000 C CNN
 F 2 "" H 17600 4500 50  0001 C CNN
 F 3 "~" H 17400 4400 50  0001 C CNN
@@
 P 17400 5350
 F 0 "Q5" V 17649 5350 50  0000 C CNN
-F 1 "Q_NMOS_DGS" V 17740 5350 50  0000 C CNN
+F 1 "BSS138" V 17740 5350 50  0000 C CNN
 F 2 "" H 17600 5450 50  0001 C CNN
 F 3 "~" H 17400 5350 50  0001 C CNN
@@
 P 17400 6300
 F 0 "Q6" V 17649 6300 50  0000 C CNN
-F 1 "Q_NMOS_DGS" V 17740 6300 50  0000 C CNN
+F 1 "BSS138" V 17740 6300 50  0000 C CNN
 F 2 "" H 17600 6400 50  0001 C CNN
 F 3 "~" H 17400 6300 50  0001 C CNN
@@
 P 18900 1400
 F 0 "Q7" V 19149 1400 50  0000 C CNN
-F 1 "Q_NMOS_DGS" V 19240 1400 50  0000 C CNN
+F 1 "BSS138" V 19240 1400 50  0000 C CNN
 F 2 "" H 19100 1500 50  0001 C CNN
 F 3 "~" H 18900 1400 50  0001 C CNN
@@
 P 18900 2400
 F 0 "Q8" V 19149 2400 50  0000 C CNN
-F 1 "Q_NMOS_DGS" V 19240 2400 50  0000 C CNN
+F 1 "BSS138" V 19240 2400 50  0000 C CNN
 F 2 "" H 19100 2500 50  0001 C CNN
 F 3 "~" H 18900 2400 50  0001 C CNN
@@
 P 18900 3400
 F 0 "Q9" V 19149 3400 50  0000 C CNN
-F 1 "Q_NMOS_DGS" V 19240 3400 50  0000 C CNN
+F 1 "BSS138" V 19240 3400 50  0000 C CNN
 F 2 "" H 19100 3500 50  0001 C CNN
 F 3 "~" H 18900 3400 50  0001 C CNN
@@
 P 18900 4400
 F 0 "Q10" V 19149 4400 50  0000 C CNN
-F 1 "Q_NMOS_DGS" V 19240 4400 50  0000 C CNN
+F 1 "BSS138" V 19240 4400 50  0000 C CNN
 F 2 "" H 19100 4500 50  0001 C CNN
 F 3 "~" H 18900 4400 50  0001 C CNN
@@
 P 18900 5350
 F 0 "Q11" V 19149 5350 50  0000 C CNN
-F 1 "Q_NMOS_DGS" V 19240 5350 50  0000 C CNN
+F 1 "BSS138" V 19240 5350 50  0000 C CNN
 F 2 "" H 19100 5450 50  0001 C CNN
 F 3 "~" H 18900 5350 50  0001 C CNN
@@
 P 18900 6300
 F 0 "Q12" V 19149 6300 50  0000 C CNN
-F 1 "Q_NMOS_DGS" V 19240 6300 50  0000 C CNN
+F 1 "BSS138" V 19240 6300 50  0000 C CNN
 F 2 "" H 19100 6400 50  0001 C CNN
 F 3 "~" H 18900 6300 50  0001 C CNN
@@
 P 20400 1400
 F 0 "Q13" V 20649 1400 50  0000 C CNN
-F 1 "Q_NMOS_DGS" V 20740 1400 50  0000 C CNN
+F 1 "BSS138" V 20740 1400 50  0000 C CNN
 F 2 "" H 20600 1500 50  0001 C CNN
 F 3 "~" H 20400 1400 50  0001 C CNN
@@
 P 20400 2400
 F 0 "Q14" V 20649 2400 50  0000 C CNN
-F 1 "Q_NMOS_DGS" V 20740 2400 50  0000 C CNN
+F 1 "BSS138" V 20740 2400 50  0000 C CNN
 F 2 "" H 20600 2500 50  0001 C CNN
 F 3 "~" H 20400 2400 50  0001 C CNN
@@
 P 20400 3400
 F 0 "Q15" V 20649 3400 50  0000 C CNN
-F 1 "Q_NMOS_DGS" V 20740 3400 50  0000 C CNN
+F 1 "BSS138" V 20740 3400 50  0000 C CNN
 F 2 "" H 20600 3500 50  0001 C CNN
 F 3 "~" H 20400 3400 50  0001 C CNN
@@
 P 20400 4400
 F 0 "Q16" V 20649 4400 50  0000 C CNN
-F 1 "Q_NMOS_DGS" V 20740 4400 50  0000 C CNN
+F 1 "BSS138" V 20740 4400 50  0000 C CNN
 F 2 "" H 20600 4500 50  0001 C CNN
 F 3 "~" H 20400 4400 50  0001 C CNN
@@
 P 20400 5350
 F 0 "Q17" V 20649 5350 50  0000 C CNN
-F 1 "Q_NMOS_DGS" V 20740 5350 50  0000 C CNN
+F 1 "BSS138" V 20740 5350 50  0000 C CNN
 F 2 "" H 20600 5450 50  0001 C CNN
 F 3 "~" H 20400 5350 50  0001 C CNN
@@
 P 20400 6300
 F 0 "Q18" V 20649 6300 50  0000 C CNN
-F 1 "Q_NMOS_DGS" V 20740 6300 50  0000 C CNN
+F 1 "BSS138" V 20740 6300 50  0000 C CNN
 F 2 "" H 20600 6400 50  0001 C CNN
 F 3 "~" H 20400 6300 50  0001 C CNN
@@
 Text Label 20150 6400 2    50   ~ 0
 M3_HALL2_3v
+$Comp
+L power:+3.3V #PWR?
+U 1 1 5F97F9E7
+P 8700 5150
+F 0 "#PWR?" H 8700 5000 50  0001 C CNN
+F 1 "+3.3V" H 8715 5323 50  0000 C CNN
+F 2 "" H 8700 5150 50  0001 C CNN
+F 3 "" H 8700 5150 50  0001 C CNN
+	1    8700 5150
+	1    0    0    -1
+$EndComp
+Wire Wire Line
+	8700 5150 9050 5150
+NoConn ~ 9050 5250
+$Comp
+L power:GND #PWR?
+U 1 1 5F9C4909
+P 8850 5800
+F 0 "#PWR?" H 8850 5550 50  0001 C CNN
+F 1 "GND" H 8855 5627 50  0000 C CNN
+F 2 "" H 8850 5800 50  0001 C CNN
+F 3 "" H 8850 5800 50  0001 C CNN
+	1    8850 5800
+	1    0    0    -1
+$EndComp
+Wire Wire Line
+	9050 5350 8850 5350
+Wire Wire Line
+	8850 5350 8850 5800
+Text Label 8700 5450 2    50   ~ 0
+RPi_SDA
+Text Label 8700 5550 2    50   ~ 0
+RPi_SCL
+Wire Wire Line
+	8700 5450 9050 5450
+Wire Wire Line
+	8700 5550 9050 5550
+NoConn ~ 9750 5250
+NoConn ~ 9750 5350
+NoConn ~ 9750 5450
+NoConn ~ 9750 5550
+Text Label 8700 5650 2    50   ~ 0
+BNO055_RST
+Wire Wire Line
+	8700 5650 9050 5650
+Text Label 3050 1950 0    50   ~ 0
+RPi_SDA
+Wire Wire Line
+	3050 1950 2900 1950
+Text Label 3050 2050 0    50   ~ 0
+RPi_SCL
+Wire Wire Line
+	3050 2050 2900 2050
+Text Label 3050 2250 0    50   ~ 0
+BNO055_RST
+Wire Wire Line
+	3050 2250 2900 2250
 $EndSCHEMATC
