File: ArmElectronics/ArmElectronics.kicad_pcb (KiCad board)
At the start: 2 copper layers, 101 x 139 mm, 90 parts, among them J1 Raspberry_Pi_2_3, J10 AH1815 Breakout, J11 AH1815 Breakout, J12 AH1815 Breakout, J13 AH1815 Breakout, J14 AH1815 Breakout, J15 AH1815 Breakout, J16 AH1815 Breakout, J17 AH1815 Breakout, J18 AH1815 Breakout, J19 AH1815 Breakout, J2 Conn_01x14, J20 AH1815 Breakout, J21 1792245, J22 PA-09, J23 PA-09, J24 PA-09, J3 Encoder Breakout, J4 RasPi Power Out, J5 12V In, J6 Batt In, J7 Batt Out, J8 BNO055 QWIIC Conn, J9 AH1815 Breakout, U1 Teensy4.1, U12 74LVC1G97, U13 74LVC1G97, U14 74LVC1G97, U15 74LVC1G97, U16 74LVC1G97, U17 74LVC1G97, U2 Pololu_2857, U3 MAX11601, U4 Pololu_2851, U5 Pololu_3730, U6 TB9051FTG, U7 TB9051FTG, U8 TB9051FTG

Commit message: Please be done now
Parts:
- moved J2 98.5 mm to (187.3, 97.3)
- moved J20 91.3 mm to (204.2, 126.2)
- moved J11 89.5 mm to (201.2, 97.6)
- moved J12 87.3 mm to (210.8, 97.6)
- moved J14 81.2 mm to (204.2, 104.6)
- moved J10 81.1 mm to (210.8, 90.4)
- moved R11 65.1 mm to (216.2, 105.5), turned to 180 degrees
- moved R10 62.5 mm to (215.2, 107.3), turned to 180 degrees
- moved J15 60.3 mm to (194.6, 111.8)
- moved C1 59.9 mm to (214.5, 109.0), turned to 180 degrees
- moved U3 55.3 mm to (216.0, 112.5), turned to 90 degrees
- moved J16 55.2 mm to (204.2, 111.8)
- moved J13 54.5 mm to (194.6, 104.6)
- moved J17 51.2 mm to (194.6, 119.0)
- moved J19 50.8 mm to (194.6, 126.2)
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Connections:
- U1 pad 32: /Hall_SW_6 -> /Stepper_Stall
- U1 pad 33: /Stepper_Stall -> /Stepper_BEMF
- U1 pad 34: /Stepper_BEMF -> /Hall_SW_4
- U1 pad 35: /Hall_SW_7 -> /Hall_SW_3
- U1 pad 36: /Hall_SW_8 -> /Hall_SW_1
- U1 pad 37: /Hall_SW_9 -> /Hall_SW_6
- U1 pad 38: /Hall_SW_10 -> /Hall_SW_8
- U1 pad 39: /Hall_SW_11 -> /Hall_SW_5
- U1 pad 4: /Hall_SW_1 -> /Hall_SW_11
- U1 pad 40: /Hall_SW_12 -> /Hall_SW_2
- U1 pad 5: /Hall_SW_2 -> /Hall_SW_12
- U1 pad 6: /Hall_SW_3 -> /Hall_SW_9
- U1 pad 7: /Hall_SW_4 -> /Hall_SW_10
- U1 pad 8: /Hall_SW_5 -> /Hall_SW_7
Routing:
- net +3V3: track 201.8 -> 356.4 mm, vias 10 -> 12
- net /Hall_SW_12: track 0.00 -> 112.2 mm
- net /Hall_SW_11: track 0.00 -> 106.0 mm
- net /Hall_SW_10: track 0.00 -> 99.2 mm
- net /Hall_SW_9: track 0.00 -> 92.9 mm
- net /RPi_GPIO12: track 0.00 -> 85.9 mm
- net /RPi_GPIO13: track 0.00 -> 81.3 mm
- net /Hall_SW_7: track 0.00 -> 78.6 mm
- net /RPi_GPIO25: track 0.00 -> 71.3 mm
- net +12V: track 0.00 -> 69.2 mm, vias 0 -> 1
- net /RPi_CS0: track 0.00 -> 64.4 mm, vias 0 -> 1
- net /RPi_GPIO24: track 0.00 -> 63.3 mm
- net /RPi_SDA: track 61.3 -> 124.3 mm, vias 2 -> 4
- net /RPi_SCL: track 57.0 -> 119.2 mm, vias 2 -> 5
- net /RPi_GPIO23: track 0.00 -> 57.9 mm
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Other:
- board text removed: "Teensy Expansion Header"
