File: ArmElectronics/ArmElectronics.kicad_pcb (KiCad board)
At the start: 2 copper layers, 101 x 139 mm, 106 parts, among them J1 Raspberry_Pi_2_3, J10 AH1815 Breakout, J11 AH1815 Breakout, J12 AH1815 Breakout, J13 AH1815 Breakout, J14 AH1815 Breakout, J15 AH1815 Breakout, J16 AH1815 Breakout, J17 AH1815 Breakout, J18 AH1815 Breakout, J19 AH1815 Breakout, J2 Conn_01x14, J20 AH1815 Breakout, J21 1792245, J22 PA-09, J23 PA-09, J24 PA-09, J25 Solenoid, J26 Stepper Alternate Connection, J27 Computer Fan, J28 Computer Fan, J3 Encoder Breakout, J4 RasPi Power Out, J5 12V In, J6 Batt In, J7 Batt Out, J8 BNO055 QWIIC Conn, J9 AH1815 Breakout, Q1 Q_NMOS_GDSD, Q2 Q_PMOS_GSD, Q3 DMMT3906, SW1 E-Stop, U1 Teensy4.1, U12 74LVC1G97, U13 74LVC1G97, U14 74LVC1G97, U15 74LVC1G97, U16 74LVC1G97, U17 74LVC1G97, U2 Pololu_2857, U3 MAX11601, U4 Pololu_2851, U5 Pololu_3730, U6 TB9051FTG, U7 TB9051FTG, U8 TB9051FTG, U9 CAT24C32

Commit message: NOT DONE FIX U3 AND SILKSCREEN
Parts:
- added G***: LOGO, ASTRA_Footprints:SHCLogoSmall, B.Cu at (68.1, 93.8)
- added G***: LOGO, ASTRA_Footprints:ATRALogo, B.Cu at (77.0, 51.4)
- U3: value MAX11601 -> MAX11607; footprint Package_TO_SOT_SMD:SOT-23-8_Handsoldering -> Package_SO:TSSOP-8_3x3mm_P0.65mm
Routing:
- net Net-(R1-Pad2): track 9.43 -> 8.37 mm
- net Net-(R3-Pad2): track 7.72 -> 6.92 mm
- net Net-(R2-Pad2): track 8.25 -> 7.51 mm
- net Net-(R4-Pad2): track 7.93 -> 7.23 mm
Other:
- board text added: "UAH SHC ASTRA Arm PCB V1.2"
- board text added: "UAH SHC ASTRA Arm PCB V1.2 Mar 2022"
- board text removed: "2020-2022"
- board text removed: "Arm Base PCB r2 UAH SHC ASTRA"

Commit message: Indicator LEDs
Parts:
- added D1: G, LED_SMD:LED_0603_1608Metric_Pad1.05x0.95mm_HandSolder, F.Cu at (72.4, 104.2)
- added D2: G, LED_SMD:LED_0603_1608Metric_Pad1.05x0.95mm_HandSolder, F.Cu at (70.4, 104.2)
- added D3: G, LED_SMD:LED_0603_1608Metric_Pad1.05x0.95mm_HandSolder, F.Cu at (105.8, 163.8)
- added D4: G, LED_SMD:LED_0603_1608Metric_Pad1.05x0.95mm_HandSolder, F.Cu at (71.4, 163.8)
- added D5: G, LED_SMD:LED_0603_1608Metric_Pad1.05x0.95mm_HandSolder, F.Cu at (68.4, 104.2)
- added R49: 10, Resistor_SMD:R_0603_1608Metric, F.Cu at (72.4, 101.0)
- added R50: 180, Resistor_SMD:R_0603_1608Metric, F.Cu at (70.4, 101.0)
- added R51: 1k, Resistor_SMD:R_0603_1608Metric, F.Cu at (109.0, 163.8)
- added R52: 3.3k, Resistor_SMD:R_0603_1608Metric, F.Cu at (68.2, 163.8)
- added R53: 180, Resistor_SMD:R_0603_1608Metric, F.Cu at (68.4, 101.0)
Connections:
- J1 pad 1: Net-(J1-Pad1) -> (no net)
- J1 pad 11: Net-(J1-Pad11) -> (no net)
- J1 pad 12: Net-(J1-Pad12) -> (no net)
- J1 pad 13: Net-(J1-Pad13) -> (no net)
- J1 pad 17: Net-(J1-Pad17) -> (no net)
- J1 pad 26: Net-(J1-Pad26) -> (no net)
- J1 pad 29: Net-(J1-Pad29) -> (no net)
- J1 pad 31: Net-(J1-Pad31) -> (no net)
- J1 pad 35: Net-(J1-Pad35) -> (no net)
- J1 pad 36: Net-(J1-Pad36) -> (no net)
- J1 pad 37: Net-(J1-Pad37) -> (no net)
- J1 pad 38: Net-(J1-Pad38) -> (no net)
- J1 pad 40: Net-(J1-Pad40) -> (no net)
- J27 pad 3: Net-(J27-Pad3) -> (no net)
- J28 pad 3: Net-(J28-Pad3) -> (no net)
- U1 pad 15: Net-(U1-Pad15) -> (no net)
- U1 pad 28: Net-(U1-Pad28) -> (no net)
- U2 pad 1: Net-(U2-Pad1) -> (no net)
- U2 pad 2: Net-(U2-Pad2) -> (no net)
- U4 pad 1: Net-(U4-Pad1) -> (no net)
- U5 pad 1: Net-(U5-Pad1) -> (no net)
- U5 pad 11: Net-(U5-Pad11) -> (no net)
- U5 pad 13: Net-(U5-Pad13) -> (no net)
- U5 pad 14: Net-(U5-Pad14) -> (no net)
- U6 pad 1: Net-(U6-Pad1) -> (no net)
- U7 pad 1: Net-(U7-Pad1) -> (no net)
- U8 pad 1: Net-(U8-Pad1) -> (no net)
- U9 pad 8: Net-(U9-Pad8) -> (no net)
Routing:
- net +3V3: track 354.9 -> 385.5 mm, vias 13 -> 14
- net /5V_RPI: track 53.4 -> 64.2 mm, vias 4 -> 6
- net +12V: track 152.6 -> 158.8 mm
- net +5V: track 307.5 -> 312.6 mm, vias 3 -> 4
- net +BATT: track 172.8 -> 174.4 mm, vias 2 -> 3
- net Net-(D4-Pad1): track 0.00 -> 1.51 mm
- net Net-(D5-Pad1): track 0.00 -> 1.50 mm
- net Net-(D3-Pad1): track 0.00 -> 1.50 mm
- net Net-(D2-Pad1): track 0.00 -> 1.50 mm
- net Net-(D1-Pad1): track 0.00 -> 1.50 mm
- net GND: vias 165 -> 166
Other:
- board text added: "3v3"
- board text added: "5v"
- board text added: "Pi"

Commit message: Ready to order?
Parts:
- moved R1 1.43 mm to (52.4, 143.3)
- moved R2 1.43 mm to (54.1, 143.3)
- moved R3 1.43 mm to (55.9, 143.3)
- moved R4 1.43 mm to (57.6, 143.3)
- moved R5 1.43 mm to (52.4, 139.8)
- moved R6 1.43 mm to (54.1, 139.8)
- moved R7 1.43 mm to (55.9, 139.8)
- moved R8 1.43 mm to (57.6, 139.8)
- moved U3 1.43 mm to (56.6, 133.8)
- moved R10 0.85 mm to (55.9, 127.9)
- moved R11 0.85 mm to (56.9, 126.2)
- moved C1 0.85 mm to (55.1, 129.7)
Routing:
- net +3V3: track 385.5 -> 387.7 mm
- net +BATT: track 174.4 -> 172.8 mm
- net +5V: track 312.6 -> 311.5 mm
- net +12V: track 158.8 -> 157.8 mm
- net /RPi_SDA: track 124.3 -> 125.1 mm
- net /RPi_SCL: track 119.5 -> 120.4 mm
- net GND: vias 166 -> 174
