File: EncoderBreakout/EncoderBreakout.sch (KiCad schematic (older format))
At the start: 8 parts, among them J1 Conn_01x06, U1 AS5047D

Commit message: Added fans
Parts:
- J1: Digikey Part Num (none) -> 455-1723-ND
Changed lines of the file:
@@
 F 2 "Connector_JST:JST_PH_S6B-PH-K_1x06_P2.00mm_Horizontal" H 3650 3900 50  0001 C CNN
 F 3 "~" H 3650 3900 50  0001 C CNN
+F 4 "455-1723-ND" H 3650 3900 50  0001 C CNN "Digikey Part Num"
 	1    3650 3900
 	-1   0    0    1
